Commit message: Using cube instead of orange. Some changes made to the reset function and the reward/goal selection and computation

File: realcomp/data/kuka_gripper_description/urdf/mustard.urdf (robot description, URDF)
Before this commit: robot mustard, 1 links, 0 joints
Links:
- link mustard: mass 2.0 -> 5.0
